File: fboard.brd (EAGLE design)
At the start: 60.9 x 51.7 mm, 29 parts, among them Q1 SL2305, U1 ATMEGA328PB-AU, U2 MPU-6050, U3 SN74HC138PW

Commit message: grounded ~g2a and ~g2b
Connections:
- net GND: now also U3.4, U3.5
Changed lines of the file:
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@@
 <drawing>
 <settings>
-<setting alwaysvectorfont="yes"/>
+<setting alwaysvectorfont="no"/>
 <setting verticaltext="up"/>
 </settings>
@@
 <vertex x="81.28" y="-11.43"/>
 </polygon>
+<contactref element="U3" pad="5"/>
+<contactref element="U3" pad="4"/>
 </signal>
 <signal name="Y0">
